Commit message: final project

File: catkin_jushanc2/src/lab2andDriver/drivers/universal_robot/ur_description/urdf/block_green.urdf (robot description, URDF)
Before this commit: robot block, 1 links, 0 joints
Links:
- link base_link: geometry collision box size=0.02 0.02 0.02; visual box size=0.02 0.02 0.02

File: catkin_jushanc2/src/lab2andDriver/drivers/universal_robot/ur_description/urdf/block_red.urdf (robot description, URDF)
Before this commit: robot block, 1 links, 0 joints
Links:
- link base_link: geometry collision box size=0.02 0.02 0.02; visual box size=0.02 0.02 0.02

File: catkin_jushanc2/src/lab2andDriver/drivers/universal_robot/ur_description/urdf/block_yellow.urdf (robot description, URDF)
Before this commit: robot block, 1 links, 0 joints
Links:
- link base_link: geometry collision box size=0.02 0.02 0.02; visual box size=0.02 0.02 0.02
